File: 16_STEP_DOWN.kicad_pcb (KiCad board)
At the start: 2 copper layers, 20.3 x 20.3 mm, 18 parts, among them J1 Conn_01x01, J2 Conn_01x01, J3 Conn_01x01, J4 Conn_01x01, J5 Conn_01x01, U1 LMR14206

Commit message: maj split librairies
Parts:
- J1, J2, J3, J4, J5: footprint Chimere:Castellated_conn -> Chimere_mods:Castellated_conn
- L1: footprint Chimere:L_Sunlord_MWSA0402S_4.2x4.4x2.0mm -> Chimere_comps:L_Sunlord_MWSA0402S_4.2x4.4x2.0mm
- U1: value LMR14206 -> LMR14203XMK
