File: 16_STEP_DOWN.sch (KiCad schematic (older format))
At the start: 18 parts, among them J1 Conn_01x01, J2 Conn_01x01, J3 Conn_01x01, J4 Conn_01x01, J5 Conn_01x01, U1 LMR14203XMK

Commit message: ajout liste compatible
Other:
- note added: "LMR14203XMK C132000\naussi compatible\nC108761\nC125906\nC193985\nC89300\nC93176"
Changed lines of the file:
@@
 	5125 1350 5125 2175
 Connection ~ 5500 2175
+Text Notes 2525 2425 0    50   ~ 0
+LMR14203XMK     C132000\naussi compatible\nC108761\nC125906\nC193985\nC89300\nC93176
 $EndSCHEMATC

Commit message: maj split librairies
Parts:
- J1, J2, J3, J4, J5: footprint Chimere:Castellated_conn -> Chimere_mods:Castellated_conn
- L1: footprint Chimere:L_Sunlord_MWSA0402S_4.2x4.4x2.0mm -> Chimere_comps:L_Sunlord_MWSA0402S_4.2x4.4x2.0mm
Changed lines of the file:
@@
 F 0 "J1" H 1880 6767 50  0000 L CNN
 F 1 "Conn_01x01" H 1880 6676 50  0000 L CNN
-F 2 "Chimere:Castellated_conn" H 1800 6725 50  0001 C CNN
+F 2 "Chimere_mods:Castellated_conn" H 1800 6725 50  0001 C CNN
 F 3 "~" H 1800 6725 50  0001 C CNN
 	1    1800 6725
@@
 F 0 "J4" H 1880 7117 50  0000 L CNN
 F 1 "Conn_01x01" H 1880 7026 50  0000 L CNN
-F 2 "Chimere:Castellated_conn" H 1800 7075 50  0001 C CNN
+F 2 "Chimere_mods:Castellated_conn" H 1800 7075 50  0001 C CNN
 F 3 "~" H 1800 7075 50  0001 C CNN
 	1    1800 7075
@@
 F 0 "J3" H 1880 6942 50  0000 L CNN
 F 1 "Conn_01x01" H 1880 6851 50  0000 L CNN
-F 2 "Chimere:Castellated_conn" H 1800 6900 50  0001 C CNN
+F 2 "Chimere_mods:Castellated_conn" H 1800 6900 50  0001 C CNN
 F 3 "~" H 1800 6900 50  0001 C CNN
 	1    1800 6900
@@
 F 0 "J2" H 3230 6792 50  0000 L CNN
 F 1 "Conn_01x01" H 3230 6701 50  0000 L CNN
-F 2 "Chimere:Castellated_conn" H 3150 6750 50  0001 C CNN
+F 2 "Chimere_mods:Castellated_conn" H 3150 6750 50  0001 C CNN
 F 3 "~" H 3150 6750 50  0001 C CNN
 	1    3150 6750
@@
 F 0 "J5" H 1880 7292 50  0000 L CNN
 F 1 "Conn_01x01" H 1880 7201 50  0000 L CNN
-F 2 "Chimere:Castellated_conn" H 1800 7250 50  0001 C CNN
+F 2 "Chimere_mods:Castellated_conn" H 1800 7250 50  0001 C CNN
 F 3 "~" H 1800 7250 50  0001 C CNN
 	1    1800 7250
@@
 F 0 "L1" V 5894 1150 50  0000 C CNN
 F 1 "MWSA0402S-100MT" V 5985 1150 50  0000 C CNN
-F 2 "Chimere:L_Sunlord_MWSA0402S_4.2x4.4x2.0mm" H 6075 1150 50  0001 C CNN
+F 2 "Chimere_comps:L_Sunlord_MWSA0402S_4.2x4.4x2.0mm" H 6075 1150 50  0001 C CNN
 F 3 "C408339" H 6075 1150 50  0001 C CNN
 	1    6075 1150
